Commit message: Several changes

File: rotors_description/urdf/iris.xacro (robot description, xacro)
@@ -20,5 +20,5 @@
   <xacro:property name="time_constant_up" value="0.0125" /> <!-- [s] -->
   <xacro:property name="time_constant_down" value="0.025" /> <!-- [s] -->
-  <xacro:property name="max_rot_velocity" value="838" /> <!-- [rad/s] -->
+  <xacro:property name="max_rot_velocity" value="1100" /> <!-- [rad/s] -->
   <xacro:property name="sin30" value="0.5" />
   <xacro:property name="cos30" value="0.866025403784" />

Commit message: Changed motor constants

File: rotors_description/urdf/iris.xacro (robot description, xacro)
@@ -18,6 +18,8 @@
   <xacro:property name="motor_constant" value="8.54858e-06" /> <!-- [kg.m/s^2] -->
   <xacro:property name="moment_constant" value="0.016" /> <!-- [m] -->
-  <xacro:property name="time_constant_up" value="0.0125" /> <!-- [s] -->
-  <xacro:property name="time_constant_down" value="0.025" /> <!-- [s] -->
+  <!-- <xacro:property name="time_constant_up" value="0.0125" />
+  <xacro:property name="time_constant_down" value="0.025" />  -->
+  <xacro:property name="time_constant_up" value="0.001" /> <!-- [s] -->
+  <xacro:property name="time_constant_down" value="0.001" /> <!-- [s] -->
   <xacro:property name="max_rot_velocity" value="1100" /> <!-- [rad/s] -->
   <xacro:property name="sin30" value="0.5" />
