Commit message: Modified launches to allow arm introduction

File: rotors_description/urdf/component_snippets.xacro (robot description, xacro)
@@ -28,5 +28,5 @@
         <frameId>${namespace}/base_link</frameId>
         <rotorVelocitySlowdownSim>${rotor_velocity_slowdown_sim}</rotorVelocitySlowdownSim>
-	<waitToRecordBag>${wait_to_record_bag}</waitToRecordBag>
+        <waitToRecordBag>${wait_to_record_bag}</waitToRecordBag>
       </plugin>
     </gazebo>
@@ -65,5 +65,5 @@
     </joint>
     <link name="${namespace}/camera_${camera_suffix}_optical_link" />
-    <joint name="${namespace}/camera_${camera_suffix}_optical_joint" type="fixed" >
+    <joint name="${namespace}/camera_${camera_suffix}_optical_joint" type="fixed">
       <origin xyz="0 0 0" rpy="${-pi/2} 0 ${-pi/2}" />
       <parent link="${namespace}/camera_${camera_suffix}_link" />
@@ -114,5 +114,5 @@
        camera. -->
   <xacro:macro name="camera_joint_macro"
-    params="namespace parent_link camera_suffix enable_visual *origin *geometry" >
+    params="namespace parent_link camera_suffix enable_visual *origin *geometry">
     <link name="${namespace}/camera_${camera_suffix}_link">
       <collision>
@@ -147,5 +147,5 @@
     params="camera_suffix horizontal_fov image_width image_height
       image_format min_distance max_distance noise_mean noise_stddev
-      baseline" >
+      baseline">
     <camera name="${camera_suffix}">
       <pose>0 ${-baseline} 0 0 0 0</pose>
@@ -191,5 +191,5 @@
     </xacro:camera_joint_macro>
     <link name="${namespace}/camera_left_optical_link" />
-    <joint name="${namespace}/camera_left_optical_joint" type="fixed" >
+    <joint name="${namespace}/camera_left_optical_joint" type="fixed">
       <origin xyz="0 0 0" rpy="${-pi/2} 0 ${-pi/2}" />
       <parent link="${namespace}/camera_left_link" />
@@ -202,17 +202,15 @@
         <!-- Here we set up the individual cameras of the stereo head. -->
         <xacro:camera_sensor_macro camera_suffix="left"
-            horizontal_fov="${horizontal_fov}" image_width="${image_width}"
-            image_height="${image_height}" image_format="${image_format}"
-            min_distance="${min_distance}" max_distance="${max_distance}"
-            noise_mean="${noise_mean}" noise_stddev="${noise_stddev}"
-            baseline="0">
-        </xacro:camera_sensor_macro>
+          horizontal_fov="${horizontal_fov}" image_width="${image_width}"
+          image_height="${image_height}" image_format="${image_format}"
+          min_distance="${min_distance}" max_distance="${max_distance}"
+          noise_mean="${noise_mean}" noise_stddev="${noise_stddev}"
+          baseline="0"></xacro:camera_sensor_macro>
         <xacro:camera_sensor_macro camera_suffix="right"
-            horizontal_fov="${horizontal_fov}" image_width="${image_width}"
-            image_height="${image_height}" image_format="${image_format}"
-            min_distance="${min_distance}" max_distance="${max_distance}"
-            noise_mean="${noise_mean}" noise_stddev="${noise_stddev}"
-            baseline="${baseline_y}">
-        </xacro:camera_sensor_macro>
+          horizontal_fov="${horizontal_fov}" image_width="${image_width}"
+          image_height="${image_height}" image_format="${image_format}"
+          min_distance="${min_distance}" max_distance="${max_distance}"
+          noise_mean="${noise_mean}" noise_stddev="${noise_stddev}"
+          baseline="${baseline_y}"></xacro:camera_sensor_macro>
         <!-- Stereo controller, setting the transforms between the two cameras. -->
         <plugin name="${namespace}_stereo_camera_controller" filename="libgazebo_ros_multicamera.so">
@@ -269,10 +267,10 @@
       <plugin name="mavlink_interface" filename="librotors_gazebo_mavlink_interface.so">
         <robotNamespace>${namespace}</robotNamespace>
-	<mavlinkControlSubTopic>${mavlink_sub_topic}</mavlinkControlSubTopic>
+        <mavlinkControlSubTopic>${mavlink_sub_topic}</mavlinkControlSubTopic>
         <imuSubTopic>${imu_sub_topic}</imuSubTopic>
         <mavlinkHilSensorPubTopic>${mavlink_pub_topic}</mavlinkHilSensorPubTopic>
-	<motorSpeedsPubTopic>${motors_speeds_pub_topic}</motorSpeedsPubTopic>
-	<gpsUpdateFreq>${gps_update_freq}</gpsUpdateFreq> <!-- Frequency of HIL GPS messages [Hz] -->
-	<rotorCount>${rotor_count}</rotorCount>
+        <motorSpeedsPubTopic>${motors_speeds_pub_topic}</motorSpeedsPubTopic>
+        <gpsUpdateFreq>${gps_update_freq}</gpsUpdateFreq> <!-- Frequency of HIL GPS messages [Hz] -->
+        <rotorCount>${rotor_count}</rotorCount>
         <!-- [Gauss] Below are the North, East, and Down components of the Earth's magnetic field at the reference location.
              The default reference location is Zurich (lat=+47.3667degN, lon=+8.5500degE, h=+500m, WGS84).
@@ -282,5 +280,5 @@
         <referenceMagEast>${reference_magnetic_field_east}</referenceMagEast>
         <referenceMagDown>${reference_magnetic_field_down}</referenceMagDown>
-	<referenceLatitude>${reference_latitude}</referenceLatitude> <!-- the initial latitude [degrees [-90, 90]] -->
+        <referenceLatitude>${reference_latitude}</referenceLatitude> <!-- the initial latitude [degrees [-90, 90]] -->
         <referenceLongitude>${reference_longitude}</referenceLongitude> <!-- the initial longitude [degrees [-180, 180]] -->
         <referenceAltitude>${reference_altitude}</referenceAltitude> <!-- the initial altitude [m] -->
@@ -300,5 +298,5 @@
       <inertial>
         <xacro:insert_block name="inertia" />
-        <mass value="${mass_imu_sensor}" />  <!-- [kg] -->
+        <mass value="${mass_imu_sensor}" /> <!-- [kg] -->
         <origin xyz="0 0 0" rpy="0 0 0" />
       </inertial>
@@ -313,5 +311,5 @@
     <gazebo>
       <plugin filename="librotors_gazebo_imu_plugin.so" name="rotors_gazebo_imu${imu_suffix}_plugin">
-      <!-- A good description of the IMU parameters can be found in the kalibr documentation:
+        <!-- A good description of the IMU parameters can be found in the kalibr documentation:
            https://github.com/ethz-asl/kalibr/wiki/IMU-Noise-Model-and-Intrinsics -->
         <robotNamespace>${namespace}</robotNamespace> <!-- (string, required): ros namespace in which the messages are published -->
@@ -344,5 +342,5 @@
       <inertial>
         <xacro:insert_block name="inertia" />
-        <mass value="${mass_odometry_sensor}" />  <!-- [kg] -->
+        <mass value="${mass_odometry_sensor}" /> <!-- [kg] -->
       </inertial>
     </link>
@@ -392,5 +390,5 @@
       <inertial>
         <xacro:insert_block name="inertia" />
-        <mass value="${mass_gps_sensor}" />  <!-- [kg] -->
+        <mass value="${mass_gps_sensor}" /> <!-- [kg] -->
         <origin xyz="0 0 0" rpy="0 0 0" />
       </inertial>
@@ -469,5 +467,5 @@
       <inertial>
         <xacro:insert_block name="inertia" />
-        <mass value="${mass_magnetometer_sensor}" />  <!-- [kg] -->
+        <mass value="${mass_magnetometer_sensor}" /> <!-- [kg] -->
         <origin xyz="0 0 0" rpy="0 0 0" />
       </inertial>
@@ -506,5 +504,5 @@
       <inertial>
         <xacro:insert_block name="inertia" />
-        <mass value="${mass_pressure_sensor}" />  <!-- [kg] -->
+        <mass value="${mass_pressure_sensor}" /> <!-- [kg] -->
         <origin xyz="0 0 0" rpy="0 0 0" />
       </inertial>
@@ -592,5 +590,5 @@
       origin_offset_x="${origin_offset_x}"
       baseline_y="${baseline_y}"
-      origin_offset_z="${origin_offset_z}" >
+      origin_offset_z="${origin_offset_z}">
       <cylinder length="0.01" radius="0.007" />
     </xacro:stereo_camera_macro>
@@ -698,6 +696,5 @@
         namespace="${namespace}" parent_link="${namespace}/vi_sensor_link"
         frame_rate="30.0" origin_offset_x="0.015" baseline_y="${0.055*2}"
-        origin_offset_z="0.0065" max_range="30.0">
-      </xacro:vi_sensor_stereo_camera_macro>
+        origin_offset_z="0.0065" max_range="30.0"></xacro:vi_sensor_stereo_camera_macro>
     </xacro:if>
     <!-- Depth Sensor -->
@@ -892,6 +889,18 @@
       reference_latitude="47.3667"
       reference_longitude="8.5500"
-      reference_altitude="500.0">
-    </xacro:mavlink_interface_macro>
+      reference_altitude="500.0"></xacro:mavlink_interface_macro>
+  </xacro:macro>
+  <!-- Macro to a torque controller to a robotic arm-->
+  <xacro:macro name="transmission_interface" params="name joint_name actuator_name">
+    <transmission name="${name}">
+      <type>transmission_interface/SimpleTransmission</type>
+      <joint name="${joint_name}">
+        <hardwareInterface>hardware_interface/EffortJointInterface</hardwareInterface>
+      </joint>
+      <actuator name="${actuator_name}">
+        <hardwareInterface>hardware_interface/EffortJointInterface</hardwareInterface>
+        <mechanicalReduction>1</mechanicalReduction>
+      </actuator>
+    </transmission>
   </xacro:macro>
 </robot>

File: rotors_description/urdf/hexacopter370.xacro (robot description, xacro)
@@ -1,9 +1,26 @@
 <?xml version="1.0"?>
-<robot name="hexarotor370" xmlns:xacro="http://ros.org/wiki/xacro">
+<!--
+  Copyright 2015 Fadri Furrer, ASL, ETH Zurich, Switzerland
+  Copyright 2015 Michael Burri, ASL, ETH Zurich, Switzerland
+  Copyright 2015 Mina Kamel, ASL, ETH Zurich, Switzerland
+  Copyright 2015 Janosch Nikolic, ASL, ETH Zurich, Switzerland
+  Copyright 2015 Markus Achtelik, ASL, ETH Zurich, Switzerland
+  Copyright 2020 Pep Marti-Saumell, IRI: CSIC-UPC, Catalunya
+  Licensed under the Apache License, Version 2.0 (the "License");
+  you may not use this file except in compliance with the License.
+  You may obtain a copy of the License at
+  http://www.apache.org/licenses/LICENSE-2.0
+  Unless required by applicable law or agreed to in writing, software
+  distributed under the License is distributed on an "AS IS" BASIS,
+  WITHOUT WARRANTIES OR CONDITIONS OF ANY KIND, either express or implied.
+  See the License for the specific language governing permissions and
+  limitations under the License.
+-->
+<robot name="hexacopter370" xmlns:xacro="http://ros.org/wiki/xacro">
   <!-- Properties -->
   <xacro:property name="namespace" value="$(arg namespace)" />
   <xacro:property name="rotor_velocity_slowdown_sim" value="10" />
   <xacro:property name="use_mesh_file" value="true" />
-  <xacro:property name="mesh_file" value="package://rotors_description/meshes/hexarotor370.dae" />
+  <xacro:property name="mesh_file" value="package://rotors_description/meshes/hexacopter370.dae" />
   <xacro:property name="mass" value="1.9828" /> <!-- [kg] -->
   <xacro:property name="body_width" value="0.40" /> <!-- [m] -->

File: rotors_description/urdf/hexacopter370_base.xacro (robot description, xacro)
@@ -17,10 +17,18 @@
   limitations under the License.
 -->
-<robot name="hexarotor370" xmlns:xacro="http://ros.org/wiki/xacro">
+<robot name="hexacopter370" xmlns:xacro="http://ros.org/wiki/xacro">
   <xacro:include filename="$(find rotors_description)/urdf/component_snippets.xacro" />
-  <!-- Instantiate hexarotor370 "mechanics" -->
-  <xacro:include filename="$(find rotors_description)/urdf/hexarotor370.xacro" />
+  <!-- Instantiate hexacopter370 "mechanics" -->
+  <xacro:include filename="$(find rotors_description)/urdf/hexacopter370.xacro" />
   <!-- Instantiate a controller. -->
   <xacro:controller_plugin_macro namespace="${namespace}" imu_sub_topic="imu" />
+  <xacro:if value="$(arg arm_enable)">
+    <xacro:include filename="$(find rotors_description)/urdf/arms/$(arg arm_name).xacro" />
+    <xacro:flying_arm_base_macro
+      namespace="${namespace}"
+      base_link="base_link"
+      origin_xyz="0.0 0.0 -0.10"
+      origin_rpy="0 0 0" />
+  </xacro:if>
   <!-- Instantiate a ROS message interface -->
   <!-- <xacro:ros_interface_plugin_macro namespace="${namespace}" />-->
