Commit message: Fixed hexxacotper model

File: rotors_description/urdf/arms/flying_arm_5.xacro (robot description, xacro)
@@ -71,5 +71,5 @@
       </visual>
     </link>
-    <gazebo reference="${namespace}/link_1">
+    <gazebo reference="${arm_namespace}/link_1">
       <mu1>0.9</mu1>
       <mu2>0.9</mu2>

File: rotors_description/urdf/hexacopter370.xacro (robot description, xacro)
@@ -23,5 +23,5 @@
   <xacro:property name="use_mesh_file" value="true" />
   <xacro:property name="mesh_file" value="package://rotors_description/meshes/hexacopter370.dae" />
-  <xacro:property name="mass" value="1.9828" /> <!-- [kg] -->
+  <xacro:property name="mass" value="1.959" /> <!-- [kg] -->
   <xacro:property name="body_width" value="0.40" /> <!-- [m] -->
   <xacro:property name="body_height" value="0.2" /> <!-- [m] -->
@@ -44,5 +44,5 @@
   <!-- Property Blocks -->
   <xacro:property name="body_inertia">
-    <inertia ixx="0.0013076" ixy="6.3281E-06" ixz="-8.4594E-06" iyy="0.0022761" iyz="1.9836E-06" izz="0.0031313" /> <!-- [kg.m^2] [kg.m^2] [kg.m^2] [kg.m^2] [kg.m^2] [kg.m^2] -->
+    <inertia ixx="0.0134943" ixy="-9.6E-06" ixz="2.82E-05" iyy="0.0141622" iyz="-7.9E-06" izz="0.0237319" /> <!-- [kg.m^2] [kg.m^2] [kg.m^2] [kg.m^2] [kg.m^2] [kg.m^2] -->
   </xacro:property>
   <!-- inertia of a single rotor, assuming it is a cuboid. Height=3mm, width=15mm -->
