Commit message: added flying_arm_3

File: rotors_description/urdf/arms/flying_arm_3.xacro (robot description, xacro)
@@ -12,5 +12,5 @@
   <xacro:property name="effort_limit_arm_link4_link5" value="0.3" />
   <xacro:property name="velocity_limit_arm_link4_link5" value="10000" />
-  <xacro:property name="arm_namespace" value="flying_arm_5" />
+  <xacro:property name="arm_namespace" value="flying_arm_3" />
   <xacro:macro name="flying_arm_base_macro" params="namespace base_link origin_xyz origin_rpy">
     <joint name="${arm_namespace}/j_base_link" type="fixed">
@@ -36,5 +36,5 @@
         <origin xyz="0 0 0" rpy="0 0 0" />
         <geometry>
-          <mesh filename="package://rotors_description/meshes/arms/flying_arm_5/base_link.dae" />
+          <mesh filename="package://rotors_description/meshes/arms/flying_arm_3/base_link.dae" />
         </geometry>
         <material name="">
@@ -64,5 +64,5 @@
         <origin xyz="0 0 0" rpy="0 0 0" />
         <geometry>
-          <mesh filename="package://rotors_description/meshes/arms/flying_arm_5/link_1.dae" />
+          <mesh filename="package://rotors_description/meshes/arms/flying_arm_3/link_1.dae" />
         </geometry>
         <material name="">
@@ -84,5 +84,5 @@
         <origin xyz="0 0 0" rpy="0 0 0" />
         <geometry>
-          <mesh filename="package://rotors_description/meshes/arms/flying_arm_5/link_2.dae" />
+          <mesh filename="package://rotors_description/meshes/arms/flying_arm_3/link_2.dae" />
         </geometry>
         <material name="">
@@ -105,12 +105,12 @@
     <link name="${arm_namespace}/link_3">
       <inertial>
-        <origin xyz="0.00020827 -0.0031223 -0.011966" rpy="0 0 0" />
-        <mass value="0.068772" />
-        <inertia ixx="6.8293E-06" ixy="4.2309E-08" ixz="1.548E-09" iyy="7.2432E-06" iyz="1.6138E-08" izz="7.1043E-06" />
+        <origin xyz="0.017465 3.6051E-08 -0.011925" rpy="0 0 0" />
+        <mass value="0.030904" />
+        <inertia ixx="1.1642E-05" ixy="1.2728E-11" ixz="-2.021E-11" iyy="2.3435E-05" iyz="-2.6426E-12" izz="1.6394E-05" />
       </inertial>
       <visual>
         <origin xyz="0 0 0" rpy="0 0 0" />
         <geometry>
-          <mesh filename="package://rotors_description/meshes/arms/flying_arm_5/link_3.dae" />
+          <mesh filename="package://rotors_description/meshes/arms/flying_arm_3/link_3.dae" />
         </geometry>
         <material name="">
@@ -130,59 +130,4 @@
       <limit lower="${- PI / 2 - 0.1}" upper="${ PI / 2 + 0.1}" effort="${effort_limit_arm_link2_link3}" velocity="${velocity_limit_arm_link2_link3}" />
       <dynamics damping="0.1" friction="0.1" />
-    </joint>
-    <link name="${arm_namespace}/link_4">
-      <inertial>
-        <origin xyz="0.026125 2.9724E-09 0.0016875" rpy="0 0 0" />
-        <mass value="0.05914" />
-        <inertia ixx="2.2712E-05" ixy="2.3256E-12" ixz="5.2509E-09" iyy="2.472E-05" iyz="3.3225E-09" izz="1.0444E-05" />
-      </inertial>
-      <visual>
-        <origin xyz="0 0 0" rpy="0 0 0" />
-        <geometry>
-          <mesh filename="package://rotors_description/meshes/arms/flying_arm_5/link_4.dae" />
-        </geometry>
-        <material name="">
-          <color rgba="0.75294 0.75294 0.75294 1" />
-        </material>
-      </visual>
-    </link>
-    <gazebo reference="${arm_namespace}/link_4">
-      <mu1>0.9</mu1>
-      <mu2>0.9</mu2>
-    </gazebo>
-    <joint name="${arm_namespace}/j_link_3_link_4" type="revolute">
-      <origin xyz="0 0 -0.011925" rpy="1.5708 0 0" />
-      <parent link="${arm_namespace}/link_3" />
-      <child link="${arm_namespace}/link_4" />
-      <axis xyz="0 0 1" />
-      <limit lower="${- PI / 2 - 0.1}" upper="${ PI / 2 + 0.1}" effort="${effort_limit_arm_link3_link4}" velocity="${velocity_limit_arm_link3_link4}" />
-      <dynamics damping="0.1" friction="0.1" />
-    </joint>
-    <link name="${arm_namespace}/link_5">
-      <inertial>
-        <origin xyz="1.7347E-18 -1.0246E-17 0.025817" rpy="0 0 0" />
-        <mass value="0.021791" />
-        <inertia ixx="7.9107E-06" ixy="1.6653E-13" ixz="2.9904E-21" iyy="1.5446E-05" iyz="-1.1963E-21" izz="1.0818E-05" />
-      </inertial>
-      <visual>
-        <origin xyz="0 0 0" rpy="0 0 0" />
-        <geometry>
-          <mesh filename="package://rotors_description/meshes/arms/flying_arm_5/link_5.dae" />
-        </geometry>
-        <material name="">
-          <color rgba="0.75294 0.75294 0.75294 1" />
-        </material>
-      </visual>
-    </link>
-    <gazebo reference="${arm_namespace}/link_5">
-      <mu1>0.9</mu1>
-      <mu2>0.9</mu2>
-    </gazebo>
-    <joint name="${arm_namespace}/j_link_4_link_5" type="revolute">
-      <origin xyz="0.034 0 -0.00025" rpy="1.5708 0 1.5708" />
-      <parent link="${arm_namespace}/link_4" />
-      <child link="${arm_namespace}/link_5" />
-      <axis xyz="0 0 1" />
-      <limit lower="${- PI /2 - 0.1}" upper="${ PI /2 + 0.1}" effort="${effort_limit_arm_link4_link5}" velocity="${velocity_limit_arm_link4_link5}" />
     </joint>
     <xacro:include filename="$(find rotors_description)/urdf/component_snippets.xacro" />
@@ -204,12 +149,4 @@
       joint_name="${arm_namespace}/j_link_2_link_3"
       actuator_name="motor3" />
-    <xacro:transmission_interface
-      name="transmission4"
-      joint_name="${arm_namespace}/j_link_3_link_4"
-      actuator_name="motor4" />
-    <xacro:transmission_interface
-      name="transmission5"
-      joint_name="${arm_namespace}/j_link_4_link_5"
-      actuator_name="motor5" />
   </xacro:macro>
 </robot>

Commit message: flying_arm_3: Firction and damping coefs

File: rotors_description/urdf/arms/flying_arm_3.xacro (robot description, xacro)
@@ -8,8 +8,4 @@
   <xacro:property name="effort_limit_arm_link2_link3" value="0.3" />
   <xacro:property name="velocity_limit_arm_link2_link3" value="10000" />
-  <xacro:property name="effort_limit_arm_link3_link4" value="0.3" />
-  <xacro:property name="velocity_limit_arm_link3_link4" value="10000" />
-  <xacro:property name="effort_limit_arm_link4_link5" value="0.3" />
-  <xacro:property name="velocity_limit_arm_link4_link5" value="10000" />
   <xacro:property name="arm_namespace" value="flying_arm_3" />
   <xacro:macro name="flying_arm_base_macro" params="namespace base_link origin_xyz origin_rpy">
@@ -39,5 +35,5 @@
         </geometry>
         <material name="">
-          <color rgba="0.75294 0.75294 0.75294 1" />
+          <color rgba="0.8471 0.6078 0.3412 1" />
         </material>
       </visual>
@@ -53,5 +49,5 @@
       <axis xyz="0 0 1" />
       <limit lower="${- PI / 2 - 0.1}" upper="${ PI / 2 + 0.1}" effort="${effort_limit_arm_bl_link1}" velocity="${velocity_limit_arm_bl_link1}" />
-      <dynamics damping="0.1" friction="0.1" />
+      <dynamics damping="0.005" friction="0.0" />
     </joint>
     <link name="${arm_namespace}/link_1">
@@ -101,5 +97,5 @@
       <axis xyz="0 0 1" />
       <limit lower="${- PI / 2 - 0.1}" upper="${ PI / 2 + 0.1}" effort="${effort_limit_arm_link1_link2}" velocity="${velocity_limit_arm_link1_link2}" />
-      <dynamics damping="0.1" friction="0.1" />
+      <dynamics damping="0.005" friction="0.0" />
     </joint>
     <link name="${arm_namespace}/link_3">
@@ -129,5 +125,5 @@
       <axis xyz="0 0 1" />
       <limit lower="${- PI / 2 - 0.1}" upper="${ PI / 2 + 0.1}" effort="${effort_limit_arm_link2_link3}" velocity="${velocity_limit_arm_link2_link3}" />
-      <dynamics damping="0.1" friction="0.1" />
+      <dynamics damping="0.005" friction="0.0" />
     </joint>
     <xacro:include filename="$(find rotors_description)/urdf/component_snippets.xacro" />
